File: PCB/logical gate/OR_gate/OR_gate.kicad_pcb (KiCad board)
At the start: 2 copper layers, 19.8 x 22.1 mm, 38 parts, among them J1 Conn_01x07, J2 Conn_01x07, Q1 P, Q10 N, Q11 P, Q12 N, Q2 N, Q3 P, Q4 N, Q5 P, Q6 N, Q7 P, Q8 N, Q9 P

Commit message: 20230309 1854
Parts:
- added Q13: N-MOS, Package_TO_SOT_SMD:SOT-23, B.Cu at (92.0, 131.4)
- added Q14: N-MOS, Package_TO_SOT_SMD:SOT-23, F.Cu at (98.9, 123.8)
- added Q15: P-MOS, Package_TO_SOT_SMD:SOT-23, F.Cu at (92.0, 127.6)
- added Q16: P-MOS, Package_TO_SOT_SMD:SOT-23, B.Cu at (92.0, 127.6)
- added Q17: N-MOS, Package_TO_SOT_SMD:SOT-23, F.Cu at (92.0, 131.4)
- added Q18: P-MOS, Package_TO_SOT_SMD:SOT-23, B.Cu at (98.9, 127.6)
- added Q19: P-MOS, Package_TO_SOT_SMD:SOT-23, F.Cu at (98.9, 127.6)
- added Q20: N-MOS, Package_TO_SOT_SMD:SOT-23, B.Cu at (98.9, 123.8)
- added Q21: P-MOS, Package_TO_SOT_SMD:SOT-23, B.Cu at (92.0, 123.8)
- added Q22: N-MOS, Package_TO_SOT_SMD:SOT-23, F.Cu at (92.0, 123.8)
- added Q23: P-MOS, Package_TO_SOT_SMD:SOT-23, B.Cu at (98.9, 131.4)
- added Q24: N-MOS, Package_TO_SOT_SMD:SOT-23, F.Cu at (98.9, 131.4)
- Q1, Q5: value P -> N-MOS
- Q10, Q12, Q2: value N -> N-MOS
- Q11, Q9: value P -> P-MOS; moved to B.Cu
- Q3, Q7: value P -> P-MOS
- Q4: value N -> P-MOS; moved to B.Cu
- Q6: value N -> P-MOS
- Q8: value N -> N-MOS; moved to B.Cu
- moved D9 92.8 mm to (96.5, 136.1), turned to 90 degrees
- moved R9 92.8 mm to (96.5, 136.1), turned to 90 degrees
- moved D11 91.2 mm to (91.4, 136.1), turned to 90 degrees
- moved R11 91.2 mm to (91.4, 136.1), turned to 90 degrees
- moved Q2 85.9 mm to (95.5, 131.4)
- moved D7 84.9 mm to (101.6, 136.1)
- moved R7 84.9 mm to (101.6, 136.1)
- moved J2 82.0 mm to (88.9, 139.7)
- moved D10 81.5 mm to (94.0, 136.1)
- moved R10 81.5 mm to (94.0, 136.1)
- moved D8 80.8 mm to (99.1, 136.1)
- moved R8 80.8 mm to (99.1, 136.1)
- moved Q6 80.4 mm to (95.5, 127.6)
- moved D12 79.7 mm to (88.9, 136.1)
- moved R12 79.7 mm to (88.9, 136.1)
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Connections:
- J1 pad 1: In6 -> B4
- J1 pad 2: In5 -> A4
- J1 pad 3: In4 -> Q3
- J1 pad 4: In3 -> Q2
- J1 pad 5: In2 -> B1
- J1 pad 6: In1 -> A1
- J2 pad 1: Out1 -> Q1
- J2 pad 2: Out2 -> A2
- J2 pad 3: Out3 -> B2
- J2 pad 4: Out4 -> A3
- J2 pad 5: Out5 -> B3
- J2 pad 6: Out6 -> Q4
- Q1 pad 1: In1 -> B1
- Q1 pad 2: +5V -> GND
- Q1 pad 3: Out1 -> Net-(Q1-Pad3)
- Q10 pad 1: In3 -> Net-(Q1-Pad3)
- Q10 pad 3: Out3 -> Q1
- Q11 pad 1: In4 -> Net-(Q11-Pad1)
- Q11 pad 3: Out4 -> Q3
- Q12 pad 1: In4 -> Net-(Q11-Pad1)
- Q12 pad 3: Out4 -> Q3
- Q2 pad 1: In1 -> B3
- Q2 pad 3: Out1 -> Net-(Q11-Pad1)
- Q3 pad 1: In5 -> A1
- Q3 pad 3: Out5 -> Net-(Q3-Pad3)
- Q4 pad 1: In5 -> B1
- Q4 pad 2: GND -> Net-(Q3-Pad3)
- Q4 pad 3: Out5 -> Net-(Q1-Pad3)
- Q5 pad 1: In2 -> A1
- Q5 pad 2: +5V -> GND
- Q5 pad 3: Out2 -> Net-(Q1-Pad3)
- Q6 pad 1: In2 -> A3
- Q6 pad 2: GND -> +5V
- Q6 pad 3: Out2 -> Net-(Q6-Pad3)
- Q7 pad 1: In6 -> B3
- Q7 pad 2: +5V -> Net-(Q6-Pad3)
- Q7 pad 3: Out6 -> Net-(Q11-Pad1)
- Q8 pad 1: In6 -> A3
- Q8 pad 3: Out6 -> Net-(Q11-Pad1)
- Q9 pad 1: In3 -> Net-(Q1-Pad3)
- Q9 pad 3: Out3 -> Q1
- R1 pad 1: In1 -> A1
- R10 pad 1: Out3 -> B2
- R11 pad 1: In4 -> A2
- R12 pad 1: Out4 -> Q1
- R2 pad 1: In5 -> B1
- R3 pad 1: Out1 -> Q2
- R4 pad 1: Out5 -> Q3
- R5 pad 1: In2 -> A4
- R6 pad 1: In6 -> B4
- R7 pad 1: Out2 -> Q4
- R8 pad 1: Out6 -> B3
- R9 pad 1: In3 -> A3
Routing:
- net Out1: track 16.0 -> 0.00 mm
- net B4: track 0.00 -> 15.6 mm, vias 0 -> 1
- net Q1: track 0.00 -> 15.5 mm, vias 0 -> 1
- net B3: track 0.00 -> 15.5 mm, vias 0 -> 1
- net Q2: track 0.00 -> 15.4 mm, vias 0 -> 1
- net In2: track 14.9 -> 0.00 mm
- net A3: track 0.00 -> 14.4 mm
- net A4: track 0.00 -> 14.4 mm
- net Net-(Q11-Pad1): track 0.00 -> 13.5 mm, vias 0 -> 3
- net In6: track 13.0 -> 0.00 mm, vias 1 -> 0
- net Out5: track 13.0 -> 0.00 mm, vias 1 -> 0
- net Q3: track 0.00 -> 13.0 mm, vias 0 -> 2
- net Out6: track 12.6 -> 0.00 mm, vias 1 -> 0
- net Out4: track 12.6 -> 0.00 mm, vias 1 -> 0
- net Out2: track 12.2 -> 0.00 mm
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Other:
- board size 19.8 x 22.1 mm -> 20.6 x 29.5 mm
- board text added: "OR CMOS"
- board text removed: "N"
- board text removed: "NOT_GATE"
